Commit message: Simplify and streamline codebase: remove redundant comments and decorative markup

File: balancing_bot.urdf (robot description, URDF)
Before this commit: robot balancing_bot, 3 links, 2 joints
Links:
- link base_link: geometry collision box size=0.08 0.18 0.26; visual box size=0.08 0.18 0.26
- link left_wheel: geometry collision cylinder length=0.025 radius=0.05; visual cylinder length=0.025 radius=0.05
- link right_wheel: geometry collision cylinder length=0.025 radius=0.05; visual cylinder length=0.025 radius=0.05
Joints:
- joint left_wheel_joint: origin xyz=0.0 0.11 0.0 rpy=0 0 0 -> xyz=0 0.11 0 rpy=0 0 0
- joint right_wheel_joint: origin xyz=0.0 -0.11 0.0 rpy=0 0 0 -> xyz=0 -0.11 0 rpy=0 0 0
